File: Circuito/dom32-touch/dom32-touch.kicad_sch (KiCad schematic)
At the start: 46 parts, among them J1 MEM2067-02-180-00-A, J2 Poste X 5, J3 MSP3218_LCD, J4 MSP3218_SD, J5 DEBUG, SW1 TactSwitch, U1 ZLDO1117QG33TADICT-ND, U2 PIC32MM0256GPM028-I-SS

Commit message: Update
Parts:
- R22: value 1K -> 33R
Connections:
- net GND: no longer R2.2, R6.2, U2.17 (TCK/RP13/RB8)
- new net: R2.2, R6.2, U2.17 (TCK/RP13/RB8)
Changed lines of the file:
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@@
   (junction (at 135.89 81.28) (diameter 0) (color 0 0 0 0)
   )
-  (junction (at 142.24 106.68) (diameter 0) (color 0 0 0 0)
-  )
   (junction (at 162.56 134.62) (diameter 0) (color 0 0 0 0)
   )
@@
     (stroke (width 0) (type default))
   )
-  (wire (pts (xy 142.24 106.68) (xy 157.48 106.68))
+  (wire (pts (xy 123.19 106.68) (xy 157.48 106.68))
     (stroke (width 0) (type default))
   )
@@
     (stroke (width 0) (type default))
   )
-  (wire (pts (xy 142.24 99.06) (xy 142.24 106.68))
+  (wire (pts (xy 142.24 99.06) (xy 142.24 125.73))
     (stroke (width 0) (type default))
   )
@@
   )
   (wire (pts (xy 154.94 148.59) (xy 139.7 148.59))
-    (stroke (width 0) (type default))
-  )
-  (wire (pts (xy 123.19 106.68) (xy 142.24 106.68))
     (stroke (width 0) (type default))
   )
@@
     )
   )
-  (symbol (lib_id "power:GND") (at 142.24 106.68 0) (unit 1)
-    (in_bom yes) (on_board yes) (dnp no)
-    (property "Reference" "#PWR010" (at 142.24 113.03 0)
-      (effects (font (size 1.27 1.27)) hide)
-    )
-    (property "Value" "GND" (at 142.367 111.0742 0)
-      (effects (font (size 1.27 1.27)) hide)
-    )
-    (property "Footprint" "" (at 142.24 106.68 0)
-      (effects (font (size 1.27 1.27)) hide)
-    )
-    (property "Datasheet" "" (at 142.24 106.68 0)
+  (symbol (lib_id "power:GND") (at 142.24 125.73 0) (unit 1)
+    (in_bom yes) (on_board yes) (dnp no)
+    (property "Reference" "#PWR010" (at 142.24 132.08 0)
+      (effects (font (size 1.27 1.27)) hide)
+    )
+    (property "Value" "GND" (at 142.367 130.1242 0)
+      (effects (font (size 1.27 1.27)) hide)
+    )
+    (property "Footprint" "" (at 142.24 125.73 0)
+      (effects (font (size 1.27 1.27)) hide)
+    )
+    (property "Datasheet" "" (at 142.24 125.73 0)
       (effects (font (size 1.27 1.27)) hide)
     )
@@
       (effects (font (size 1.27 1.27)))
     )
-    (property "Value" "1K" (at 71.9836 127 90)
-      (effects (font (size 1.27 1.27)))
-    )
+    (property "Value" "33R" (at 71.9836 127 90)
+      (effects (font (size 1.27 1.27)))
+    )
