File: Circuito/dom32-touch.kicad_pcb (KiCad board)
At the start: 2 copper layers, 60 x 44 mm, 44 parts, among them J1 Poste X 5, J2 277-1667-ND, J3 CF4240FH0R0-05-NH, J4 DEBUG & Buzzer, J5 MEM2067-02-180-00-A, Q1 BC548, SW1 TactSwitch, U1 ZLDO1117QG33TADICT-ND, U2 PIC32MM0256GPM028-I-SS, U3 1965-ESP-WROOM-02D-N4CT-ND

Commit message: Circuito Impreso
Circuito Impreso
Parts:
- added D10: Cortesia, Diode_SMD:D_0805_2012Metric_Pad1.15x1.40mm_HandSolder, F.Cu at (131.0, 113.0)
- added D11: Cortesia, Diode_SMD:D_0805_2012Metric_Pad1.15x1.40mm_HandSolder, F.Cu at (131.0, 99.0)
- added D12: Cortesia, Diode_SMD:D_0805_2012Metric_Pad1.15x1.40mm_HandSolder, F.Cu at (131.0, 85.0)
- added D5: Power Ok, Diode_SMD:D_0805_2012Metric_Pad1.15x1.40mm_HandSolder, F.Cu at (187.0, 93.0)
- added D6: Error, Diode_SMD:D_0805_2012Metric_Pad1.15x1.40mm_HandSolder, F.Cu at (187.0, 85.0)
- added D7: Cortesia, Diode_SMD:D_0805_2012Metric_Pad1.15x1.40mm_HandSolder, F.Cu at (131.0, 92.0)
- added D8: Cortesia, Diode_SMD:D_0805_2012Metric_Pad1.15x1.40mm_HandSolder, F.Cu at (131.0, 78.0)
- added D9: Cortesia, Diode_SMD:D_0805_2012Metric_Pad1.15x1.40mm_HandSolder, F.Cu at (131.0, 106.0)
- added R20: 1K, Resistor_SMD:R_0805_2012Metric_Pad1.20x1.40mm_HandSolder, F.Cu at (184.0, 93.0)
- added R21: 1K, Resistor_SMD:R_0805_2012Metric_Pad1.20x1.40mm_HandSolder, F.Cu at (184.0, 85.0)
- added R22: 1K, Resistor_SMD:R_0805_2012Metric_Pad1.20x1.40mm_HandSolder, F.Cu at (155.0, 116.0)
- C11, C8: value 100uf / 16v -> 100uf / 25v; footprint Capacitor_THT:CP_Radial_D6.3mm_P2.50mm -> Capacitor_SMD:CP_Elec_6.3x7.7
- C4: footprint Capacitor_THT:CP_Radial_D8.0mm_P5.00mm -> Capacitor_SMD:CP_Elec_6.3x7.7
- C5, C9: footprint Capacitor_THT:CP_Radial_D6.3mm_P2.50mm -> Capacitor_SMD:CP_Elec_6.3x7.7
- Q1: footprint Package_TO_SOT_THT:TO-92_Inline -> Package_TO_SOT_SMD:SOT-23
- R10, R11, R12, R13, R14, R15, R16, R17, R18, R19, R9, U2, U3: moved to B.Cu
- SW1: footprint Button_Switch_THT:SW_PUSH_6mm_H5mm -> Button_Switch_SMD:SW_Push_1P1T_NO_6x6mm_H9.5mm
- moved R9 145.7 mm to (178.8, 97.5), turned to -90 degrees
- moved C1 144.9 mm to (178.0, 108.0), turned to 90 degrees
- moved R10 142.0 mm to (176.2, 97.5), turned to -90 degrees
- moved R15 140.6 mm to (170.5, 104.5), turned to 90 degrees
- moved C5 139.6 mm to (172.0, 86.0), turned to 90 degrees
- moved R11 138.4 mm to (173.8, 97.5), turned to -90 degrees
- moved C3 135.8 mm to (168.0, 112.0), turned to -90 degrees
- moved C9 134.3 mm to (163.0, 112.0), turned to -90 degrees
- moved R14 132.5 mm to (168.0, 104.5), turned to 90 degrees
- moved C6 132.3 mm to (177.0, 96.5)
- moved R13 131.9 mm to (165.5, 104.5), turned to 90 degrees
- moved R12 131.4 mm to (163.0, 104.5), turned to 90 degrees
- moved R7 130.3 mm to (155.0, 113.0)
- moved R2 129.2 mm to (161.8, 85.8)
- moved R6 128.5 mm to (162.0, 95.8), turned to 180 degrees
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Routing:
- net Net-(D3-K): track 0.00 -> 128.8 mm, vias 0 -> 3
- net Net-(U2-PGEC3/RP18/RC9): track 0.00 -> 83.5 mm, vias 0 -> 1
- net Net-(C1-Pad1): track 0.00 -> 65.8 mm, vias 0 -> 2
- net Net-(D4-K): track 0.00 -> 65.5 mm, vias 0 -> 1
- net Net-(U1-VO): track 0.00 -> 62.9 mm
- net GND: track 0.00 -> 42.6 mm, vias 0 -> 41
- net Net-(J1-Pin_4): track 0.00 -> 42.2 mm, vias 0 -> 2
- net Net-(J3-Pin_25): track 0.00 -> 37.8 mm, vias 0 -> 2
- net Net-(J3-Pin_26): track 0.00 -> 37.2 mm, vias 0 -> 3
- net Net-(D1-K): track 0.00 -> 36.6 mm
- net Net-(J1-Pin_5): track 0.00 -> 35.2 mm, vias 0 -> 2
- net Net-(J5-DAT3/CD): track 0.00 -> 33.4 mm, vias 0 -> 1
- net Net-(D10-A): track 0.00 -> 33.2 mm
- net Net-(J1-Pin_1): track 0.00 -> 32.5 mm, vias 0 -> 1
- net Net-(J5-DAT0): track 0.00 -> 32.4 mm, vias 0 -> 1
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- added copper zone on B.Cu, net GND
Other:
- rule pad_to_mask_clearance: 0 -> 0.051
- board text added: "+"
- board text added: "-"

Commit message: DRC Ok
DRC Ok
Routing:
- net GND: track 42.6 -> 60.7 mm, vias 41 -> 44
- net Net-(D3-K): track 128.8 -> 136.8 mm
- net Net-(Q1-B): track 18.4 -> 14.5 mm
- net Net-(J5-DAT3/CD): track 33.4 -> 36.8 mm
- net Net-(J5-CLK): track 31.1 -> 34.2 mm
- net Net-(J5-DAT0): track 32.4 -> 35.2 mm
- net Net-(U2-D+/RB11): track 12.3 -> 14.2 mm
- net Net-(U2-PGEC3/RP18/RC9): track 83.5 -> 81.9 mm
- net Net-(J5-CMD): track 23.5 -> 24.9 mm
- net Net-(C1-Pad1): track 65.8 -> 64.6 mm
- net Net-(U2-RP15/RB13): track 9.24 -> 10.4 mm
- net Net-(U3-TXD): track 8.78 -> 9.91 mm
- net Net-(J3-Pin_35): track 26.5 -> 25.6 mm
- net Net-(U3-RXD): track 6.51 -> 7.23 mm
- added copper zone on F.Cu, net (none)
