File: Circuito/dom32-touch.kicad_pcb (KiCad board)
At the start: 2 copper layers, 60 x 44 mm, 55 parts, among them J1 Poste X 5, J2 277-1667-ND, J3 CF4240FH0R0-05-NH, J4 DEBUG & Buzzer, J5 MEM2067-02-180-00-A, Q1 BC548, SW1 TactSwitch, U1 ZLDO1117QG33TADICT-ND, U2 PIC32MM0256GPM028-I-SS, U3 1965-ESP-WROOM-02D-N4CT-ND

Commit message: Update
Update
Other:
- board text added: "Buzzer"
- board text added: "Display"
- board text added: "Dom32 Touch"
- board text added: "HECHO EN ARGENTINA"
- board text added: "RESET"
Changed lines of the file:
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@@
     (property "ki_keywords" "cap capacitor")
     (attr smd)
-    (fp_text reference "C2" (at 3 0) (layer "F.SilkS")
+    (fp_text reference "C2" (at 0.25 2) (layer "F.SilkS")
         (effects (font (size 1 1) (thickness 0.15)))
     )
@@
     (property "ki_keywords" "R res resistor")
     (attr smd)
-    (fp_text reference "R4" (at -3 0) (layer "F.SilkS")
+    (fp_text reference "R4" (at -5.75 0) (layer "F.SilkS")
         (effects (font (size 1 1) (thickness 0.15)))
     )
@@
     (property "ki_keywords" "LED diode")
     (attr smd)
-    (fp_text reference "D7" (at 0 -1.65 90) (layer "F.SilkS")
+    (fp_text reference "D7" (at 0 -1.75 90) (layer "F.SilkS")
         (effects (font (size 1 1) (thickness 0.15)))
     )
@@
     (property "ki_keywords" "LED diode")
     (attr smd)
-    (fp_text reference "D9" (at 0 -1.65 90) (layer "F.SilkS")
+    (fp_text reference "D9" (at 0 -1.75 90) (layer "F.SilkS")
         (effects (font (size 1 1) (thickness 0.15)))
     )
@@
     (property "ki_keywords" "LED diode")
     (attr smd)
-    (fp_text reference "D8" (at 0 -1.65 90) (layer "F.SilkS")
+    (fp_text reference "D8" (at -0.025 -1.75 90) (layer "F.SilkS")
         (effects (font (size 1 1) (thickness 0.15)))
     )
@@
     (property "ki_keywords" "LED diode")
     (attr smd)
-    (fp_text reference "D6" (at 3 0 90) (layer "F.SilkS")
+    (fp_text reference "D6" (at 3 -0.25 90) (layer "F.SilkS")
         (effects (font (size 1 1) (thickness 0.15)))
     )
@@
     (property "ki_keywords" "LED diode")
     (attr smd)
-    (fp_text reference "D10" (at 0 -1.65 90) (layer "F.SilkS")
+    (fp_text reference "D10" (at 0 -1.75 90) (layer "F.SilkS")
         (effects (font (size 1 1) (thickness 0.15)))
     )
@@
     (property "ki_keywords" "LED diode")
     (attr smd)
-    (fp_text reference "D11" (at 0 -1.65 90) (layer "F.SilkS")
+    (fp_text reference "D11" (at 0 -1.75 90) (layer "F.SilkS")
         (effects (font (size 1 1) (thickness 0.15)))
     )
@@
     (property "ki_keywords" "cap capacitor")
     (attr smd)
-    (fp_text reference "C4" (at 0 0 90) (layer "F.SilkS")
+    (fp_text reference "C4" (at 4.5 2.5 -180) (layer "F.SilkS")
         (effects (font (size 1 1) (thickness 0.15)))
     )
@@
     (property "ki_keywords" "LED diode")
     (attr smd)
-    (fp_text reference "D12" (at 0 -1.65 90) (layer "F.SilkS")
+    (fp_text reference "D12" (at 0 -1.75 90) (layer "F.SilkS")
         (effects (font (size 1 1) (thickness 0.15)))
     )
@@
     (property "ki_keywords" "cap capacitor")
     (attr smd)
-    (fp_text reference "C3" (at 4.5375 7.75 -180) (layer "F.SilkS")
+    (fp_text reference "C3" (at 3.0375 0 -180) (layer "F.SilkS")
         (effects (font (size 1 1) (thickness 0.15)))
     )
@@
     (property "ki_keywords" "cap capacitor")
     (attr smd)
-    (fp_text reference "C9" (at 0 0 90) (layer "F.SilkS")
+    (fp_text reference "C9" (at 4.5 2.75 -180) (layer "F.SilkS")
         (effects (font (size 1 1) (thickness 0.15)))
     )
@@
     (property "ki_keywords" "LED diode")
     (attr smd)
-    (fp_text reference "D5" (at 3 0 90) (layer "F.SilkS")
+    (fp_text reference "D5" (at 3 -0.25 90) (layer "F.SilkS")
         (effects (font (size 1 1) (thickness 0.15)))
     )
@@
   (gr_line (start 189.65 117.83) (end 129.65 117.83)
     (stroke (width 0.1) (type default)) (layer "Edge.Cuts"))
-  (gr_text "-" (at 189.25 97.25 90) (layer "F.SilkS")
-    (effects (font (size 1 1) (thickness 0.15)) (justify left bottom))
+  (gr_text "Dom32\nTouch" (at 183.25 113.25) (layer "B.Cu")
+    (effects (font (size 1.5 1.5) (thickness 0.3) bold) (justify left bottom mirror))
+  )
+  (gr_text "HECHO EN ARGENTINA" (at 134.75 82.75 90) (layer "B.Cu")
+    (effects (font (size 1.5 1.5) (thickness 0.3) bold) (justify left bottom mirror))
+  )
+  (gr_text "Display" (at 147 92.5 90) (layer "B.SilkS")
+    (effects (font (size 1 1) (thickness 0.15)) (justify left bottom mirror))
+  )
+  (gr_text "Buzzer" (at 140.75 79.5) (layer "B.SilkS")
+    (effects (font (size 1 1) (thickness 0.15)) (justify left bottom mirror))
+  )
+  (gr_text "-" (at 189.5 98 90) (layer "F.SilkS")
+    (effects (font (size 2 2) (thickness 0.15)) (justify left bottom))
+  )
+  (gr_text "+" (at 187 110) (layer "F.SilkS")
+    (effects (font (size 2 2) (thickness 0.15)) (justify left bottom))
   )
-  (gr_text "+" (at 188.25 109.75) (layer "F.SilkS")
+  (gr_text "RESET" (at 178.25 115.75 90) (layer "F.SilkS")
     (effects (font (size 1 1) (thickness 0.15)) (justify left bottom))
   )

Commit message: Fabricacion
Fabricacion
Parts:
- C4: value 1000uf / 25v -> 100uf / 25v
- D10, D11, D12, D7, D8, D9: value Cortesia -> Led SMD Azul
- D5: value Power Ok -> Led SMD Verde
- D6: value Error -> Led SMD Rojo
Changed lines of the file:
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@@
         (effects (font (size 1 1) (thickness 0.15)))
     )
-    (fp_text value "Cortesia" (at 0 1.65 90) (layer "F.Fab")
+    (fp_text value "Led SMD Azul" (at 0 1.65 90) (layer "F.Fab")
         (effects (font (size 1 1) (thickness 0.15)))
     )
@@
         (effects (font (size 1 1) (thickness 0.15)))
     )
-    (fp_text value "Cortesia" (at 0 1.65 90) (layer "F.Fab")
+    (fp_text value "Led SMD Azul" (at 0 1.65 90) (layer "F.Fab")
         (effects (font (size 1 1) (thickness 0.15)))
     )
@@
         (effects (font (size 1 1) (thickness 0.15)))
     )
-    (fp_text value "Cortesia" (at 0 1.65 90) (layer "F.Fab")
+    (fp_text value "Led SMD Azul" (at 0 1.65 90) (layer "F.Fab")
         (effects (font (size 1 1) (thickness 0.15)))
     )
@@
         (effects (font (size 1 1) (thickness 0.15)))
     )
-    (fp_text value "Error" (at 0 1.65 90) (layer "F.Fab")
+    (fp_text value "Led SMD Rojo" (at 0 1.65 90) (layer "F.Fab")
         (effects (font (size 1 1) (thickness 0.15)))
     )
@@
         (effects (font (size 1 1) (thickness 0.15)))
     )
-    (fp_text value "Cortesia" (at 0 1.65 90) (layer "F.Fab")
+    (fp_text value "Led SMD Azul" (at 0 1.65 90) (layer "F.Fab")
         (effects (font (size 1 1) (thickness 0.15)))
     )
@@
         (effects (font (size 1 1) (thickness 0.15)))
     )
-    (fp_text value "Cortesia" (at 0 1.65 90) (layer "F.Fab")
+    (fp_text value "Led SMD Azul" (at 0 1.65 90) (layer "F.Fab")
         (effects (font (size 1 1) (thickness 0.15)))
     )
@@
         (effects (font (size 1 1) (thickness 0.15)))
     )
-    (fp_text value "1000uf / 25v" (at 0 4.35 90) (layer "F.Fab")
+    (fp_text value "100uf / 25v" (at 0 4.35 90) (layer "F.Fab")
         (effects (font (size 1 1) (thickness 0.15)))
     )
@@
         (effects (font (size 1 1) (thickness 0.15)))
     )
-    (fp_text value "Cortesia" (at 0 1.65 90) (layer "F.Fab")
+    (fp_text value "Led SMD Azul" (at 0 1.65 90) (layer "F.Fab")
         (effects (font (size 1 1) (thickness 0.15)))
     )
@@
         (effects (font (size 1 1) (thickness 0.15)))
     )
-    (fp_text value "Power Ok" (at 0 1.65 90) (layer "F.Fab")
-        (effects (font (size 1 1) (thickness 0.15)))
-    )
+    (fp_text value "Led SMD Verde" (at 0 1.65 90) (layer "F.Fab")
+        (effects (font (size 1 1) (thickness 0.15)))
+    )
